File: Kicad/osc_input.sch (KiCad schematic (older format))
At the start: 20 parts, among them P1 CONN_01X04, P2 CONN_01X03, Q1 BC547b, Q2 BC547b, U1 LM2931A

Commit message: Kicad: Updated schematics to use kicad embedded spice simulator.
Parts:
- DM1, DP1: Spice_Lib_File (none) -> spice_models/1N4007.mod; Spice_Model (none) -> 1n4007; Spice_Netlist_Enabled (none) -> Y; Spice_Primitive (none) -> D
- P1: Spice_Lib_File (none) -> spice_models/CONN_01x04.mod; Spice_Model (none) -> CONN_01x04; Spice_Netlist_Enabled (none) -> Y; Spice_Primitive (none) -> X
- P2: Spice_Lib_File (none) -> spice_models/CONN_01x03.mod; Spice_Model (none) -> CONN_01x03; Spice_Netlist_Enabled (none) -> Y; Spice_Primitive (none) -> X
- Q1: Spice_Lib_File (none) -> spice_models/BC547B.mod; Spice_Model (none) -> bc547b; Spice_Netlist_Enabled (none) -> Y; Spice_Primitive (none) -> Q
- U1: Spice_Lib_File (none) -> spice_models/LM2931A.mod; Spice_Model (none) -> LM2931A; Spice_Netlist_Enabled (none) -> Y; Spice_Primitive (none) -> X
Other:
- note added: ".include spice_models/1N4007.mod\n.include spice_models/BC547B.mod\n.include spice_models/LM2931A.mod\n.include spice_models/CONN_01x03.mod\n.include spice_models/CONN_01x04.mod\n.include spice_models/inputs.mod\n.tran 1u 5m 4m"
- note removed: "-PSPICE \n.include spice_models/1N4007.mod\n.include spice_models/BC547B.mod\n.include spice_models/LM2931A.mod\n.include spice_models/CONN_01x03.mod\n.include spice_models/CONN_01x04.mod\nVIN1 VIN1 GND SIN(0 50 1k)\nVIN2 VIN2 GND SIN(0 50 1k)\nVCC VCC GND 4.83V\n"
Changed lines of the file:
@@
 LIBS:valves
 LIBS:boul51
+LIBS:osc_input-cache
 EELAYER 26 0
 EELAYER END
@@
 $EndComp
 $Comp
-L BC547 Q1
-U 1 1 5521824E
-P 4650 4450
-F 0 "Q1" H 4650 4301 40  0000 R CNN
-F 1 "BC547b" H 4650 4600 40  0000 R CNN
-F 2 "boul51:TO-92_1" H 4550 4552 29  0001 C CNN
-F 3 "" H 4650 4450 60  0000 C CNN
-	1    4650 4450
-	1    0    0    -1
-$EndComp
-$Comp
 L R RE1
 U 1 1 55218DEE
@@
 	4300 2200 4300 2100
 Text Notes 750  3000 0    60   ~ 0
--PSPICE \n.include spice_models/1N4007.mod\n.include spice_models/BC547B.mod\n.include spice_models/LM2931A.mod\n.include spice_models/CONN_01x03.mod\n.include spice_models/CONN_01x04.mod\nVIN1 VIN1 GND SIN(0 50 1k)\nVIN2 VIN2 GND SIN(0 50 1k)\nVCC VCC GND 4.83V\n
+.include spice_models/1N4007.mod\n.include spice_models/BC547B.mod\n.include spice_models/LM2931A.mod\n.include spice_models/CONN_01x03.mod\n.include spice_models/CONN_01x04.mod\n.include spice_models/inputs.mod\n.tran 1u 5m 4m
 Text GLabel 4300 4600 3    60   Input ~ 0
 VB1
@@
 Wire Wire Line
 	4300 3500 4300 3700
-Connection ~ 4550 2200
-Connection ~ 4300 2200
 Wire Wire Line
 	4750 4750 4950 4750
@@
 F 2 "TO_SOT_Packages_THT:TO-220_Neutral123_Vertical" H 4250 2700 30  0001 C CIN
 F 3 "" H 4250 2600 60  0000 C CNN
+F 4 "X" H 4250 2600 60  0001 C CNN "Spice_Primitive"
+F 5 "LM2931A" H 4250 2600 60  0001 C CNN "Spice_Model"
+F 6 "Y" H 4250 2600 60  0001 C CNN "Spice_Netlist_Enabled"
+F 7 "spice_models/LM2931A.mod" H 4250 2600 60  0001 C CNN "Spice_Lib_File"
 	1    4250 2600
 	0    1    1    0
 $EndComp
-Wire Wire Line
-	3900 4450 4500 4450
 Connection ~ 3450 3000
 Connection ~ 3450 3400
@@
 Wire Wire Line
 	4500 3900 4500 5000
-Connection ~ 4450 4450
 $Comp
 L GND #PWR011
@@
 	1    0    0    -1
 $EndComp
-Connection ~ 5350 1950
 Wire Wire Line
 	5450 2300 5750 2300
@@
 F 2 "boul51:Diode-DO41" H 4500 3750 60  0001 C CNN
 F 3 "" H 4500 3750 60  0000 C CNN
+F 4 "D" H 4500 3750 60  0001 C CNN "Spice_Primitive"
+F 5 "1n4007" H 4500 3750 60  0001 C CNN "Spice_Model"
+F 6 "Y" H 4500 3750 60  0001 C CNN "Spice_Netlist_Enabled"
+F 7 "spice_models/1N4007.mod" H 4500 3750 60  0001 C CNN "Spice_Lib_File"
 	1    4500 3750
 	0    -1   -1   0
@@
 F 2 "boul51:Diode-DO41" H 4500 5150 60  0001 C CNN
 F 3 "" H 4500 5150 60  0000 C CNN
+F 4 "D" H 4500 5150 60  0001 C CNN "Spice_Primitive"
+F 5 "1n4007" H 4500 5150 60  0001 C CNN "Spice_Model"
+F 6 "Y" H 4500 5150 60  0001 C CNN "Spice_Netlist_Enabled"
+F 7 "spice_models/1N4007.mod" H 4500 5150 60  0001 C CNN "Spice_Lib_File"
 	1    4500 5150
 	0    -1   -1   0
@@
 F 2 "boul51:PinHeader_x4" H 2700 4000 50  0001 C CNN
 F 3 "" H 2700 4000 50  0000 C CNN
+F 4 "X" H 2700 4000 60  0001 C CNN "Spice_Primitive"
+F 5 "CONN_01x04" H 2700 4000 60  0001 C CNN "Spice_Model"
+F 6 "Y" H 2700 4000 60  0001 C CNN "Spice_Netlist_Enabled"
+F 7 "spice_models/CONN_01x04.mod" H 2700 4000 60  0001 C CNN "Spice_Lib_File"
 	1    2700 4000
 	-1   0    0    1
@@
 F 2 "boul51:PinHeader_x3" H 5950 2300 50  0001 C CNN
 F 3 "" H 5950 2300 50  0000 C CNN
+F 4 "X" H 5950 2300 60  0001 C CNN "Spice_Primitive"
+F 5 "CONN_01x03" H 5950 2300 60  0001 C CNN "Spice_Model"
+F 6 "Y" H 5950 2300 60  0001 C CNN "Spice_Netlist_Enabled"
+F 7 "spice_models/CONN_01x03.mod" H 5950 2300 60  0001 C CNN "Spice_Lib_File"
 	1    5950 2300
 	1    0    0    -1
@@
 Wire Wire Line
 	3450 3350 3450 3400
+Connection ~ 4300 2200
+$Comp
+L BC547 Q1
+U 1 1 5521824E
+P 4650 4450
+F 0 "Q1" H 4650 4301 40  0000 R CNN
+F 1 "BC547b" H 4650 4600 40  0000 R CNN
+F 2 "boul51:TO-92_1" H 4550 4552 29  0001 C CNN
+F 3 "" H 4650 4450 60  0000 C CNN
+F 4 "Q" H 4650 4450 60  0001 C CNN "Spice_Primitive"
+F 5 "bc547b" H 4650 4450 60  0001 C CNN "Spice_Model"
+F 6 "Y" H 4650 4450 60  0001 C CNN "Spice_Netlist_Enabled"
+F 7 "spice_models/BC547B.mod" H 4650 4450 60  0001 C CNN "Spice_Lib_File"
+	1    4650 4450
+	1    0    0    -1
+$EndComp
+Wire Wire Line
+	3900 4450 4500 4450
+Connection ~ 4450 4450
 $EndSCHEMATC
